File: avionics-hw27-kiwi.kicad_sch (KiCad schematic)
At the start: 0 parts

Commit message: top level schematic hierarchy made
added schematic hierarchy pages and imported MCU part. placed MCU on its page
Other:
- added sheet LED and Button (LEDandButton.kicad_sch)
- added sheet MCU (mcu.kicad_sch)
- added sheet Power (powerkicad_sch.kicad_sch)
- added sheet RF Transciever (RF.kicad_sch)
Changed lines of the file:
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@@
 	(generator_version "10.0")
 	(paper "A4")
+	(sheet
+		(at 55.88 90.17)
+		(size 44.45 29.21)
+		(exclude_from_sim no)
+		(in_bom yes)
+		(on_board yes)
+		(dnp no)
+		(fields_autoplaced yes)
+		(stroke
+			(width 0.1524)
+			(type solid)
+		)
+		(fill
+			(color 0 0 0 0)
+		)
+		(property "Sheetname" "LED and Button"
+			(at 55.88 89.4584 0)
+			(show_name no)
+			(do_not_autoplace no)
+			(effects
+				(font
+					(size 1.27 1.27)
+				)
+				(justify left bottom)
+			)
+		)
+		(property "Sheetfile" "LEDandButton.kicad_sch"
+			(at 55.88 119.9646 0)
+			(show_name no)
+			(do_not_autoplace no)
+			(effects
+				(font
+					(size 1.27 1.27)
+				)
+				(justify left top)
+			)
+		)
+		(instances
+			(project "avionics-hw27-kiwi"
+				(path "/b8c2db8f-1b36-44ff-a894-811d925da4bc"
+					(page "4")
+				)
+			)
+		)
+	)
+	(sheet
+		(at 55.88 54.61)
+		(size 44.45 26.67)
+		(exclude_from_sim no)
+		(in_bom yes)
+		(on_board yes)
+		(dnp no)
+		(fields_autoplaced yes)
+		(stroke
+			(width 0.1524)
+			(type solid)
+		)
+		(fill
+			(color 0 0 0 0)
+		)
+		(property "Sheetname" "Power"
+			(at 55.88 53.8984 0)
+			(show_name no)
+			(do_not_autoplace no)
+			(effects
+				(font
+					(size 1.27 1.27)
+				)
+				(justify left bottom)
+			)
+		)
+		(property "Sheetfile" "powerkicad_sch.kicad_sch"
+			(at 55.88 81.8646 0)
+			(show_name no)
+			(do_not_autoplace no)
+			(effects
+				(font
+					(size 1.27 1.27)
+				)
+				(justify left top)
+			)
+		)
+		(instances
+			(project "avionics-hw27-kiwi"
+				(path "/b8c2db8f-1b36-44ff-a894-811d925da4bc"
+					(page "2")
+				)
+			)
+		)
+	)
+	(sheet
+		(at 110.49 88.9)
+		(size 40.64 30.48)
+		(exclude_from_sim no)
+		(in_bom yes)
+		(on_board yes)
+		(dnp no)
+		(fields_autoplaced yes)
+		(stroke
+			(width 0.1524)
+			(type solid)
+		)
+		(fill
+			(color 0 0 0 0)
+		)
+		(property "Sheetname" "RF Transciever"
+			(at 110.49 88.1884 0)
+			(show_name no)
+			(do_not_autoplace no)
+			(effects
+				(font
+					(size 1.27 1.27)
+				)
+				(justify left bottom)
+			)
+		)
+		(property "Sheetfile" "RF.kicad_sch"
+			(at 110.49 119.9646 0)
+			(show_name no)
+			(do_not_autoplace no)
+			(effects
+				(font
+					(size 1.27 1.27)
+				)
+				(justify left top)
+			)
+		)
+		(instances
+			(project "avionics-hw27-kiwi"
+				(path "/b8c2db8f-1b36-44ff-a894-811d925da4bc"
+					(page "5")
+				)
+			)
+		)
+	)
+	(sheet
+		(at 110.49 54.61)
+		(size 39.37 26.67)
+		(exclude_from_sim no)
+		(in_bom yes)
+		(on_board yes)
+		(dnp no)
+		(fields_autoplaced yes)
+		(stroke
+			(width 0.1524)
+			(type solid)
+		)
+		(fill
+			(color 0 0 0 0)
+		)
+		(property "Sheetname" "MCU"
+			(at 110.49 53.8984 0)
+			(show_name no)
+			(do_not_autoplace no)
+			(effects
+				(font
+					(size 1.27 1.27)
+				)
+				(justify left bottom)
+			)
+		)
+		(property "Sheetfile" "mcu.kicad_sch"
+			(at 110.49 81.8646 0)
+			(show_name no)
+			(do_not_autoplace no)
+			(effects
+				(font
+					(size 1.27 1.27)
+				)
+				(justify left top)
+			)
+		)
+		(instances
+			(project "avionics-hw27-kiwi"
+				(path "/b8c2db8f-1b36-44ff-a894-811d925da4bc"
+					(page "3")
+				)
+			)
+		)
+	)
 	(sheet_instances
 		(path "/"
