File: Detonator_Side/RF_Antenna.kicad_sch (KiCad schematic)
At the start: 1 part

Commit message: Added RF footprint
Parts:
- removed U2: (no value), Package_DFN_QFN:QFN-24-1EP_5x5mm_P0.65mm_EP3.25x3.25mm, symbol Argus-Miscellaneous:E22-900M30S-SX1262
Changed lines of the file:
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@@
 	(generator_version "10.0")
 	(paper "A4")
-	(symbol
-		(lib_id "Argus-Miscellaneous:E22-900M30S-SX1262")
-		(at 138.43 76.2 0)
-		(unit 1)
-		(body_style 1)
-		(exclude_from_sim no)
-		(in_bom yes)
-		(on_board yes)
-		(in_pos_files yes)
-		(dnp no)
-		(fields_autoplaced yes)
-		(property "Reference" "U2"
-			(at 139.065 77.47 0)
-			(show_name no)
-			(do_not_autoplace no)
-			(effects
-				(font
-					(size 1.27 1.27)
-				)
-			)
-		)
-		(property "Value" ""
-			(at 138.43 76.2 0)
-			(show_name no)
-			(do_not_autoplace no)
-			(effects
-				(font
-					(size 1.27 1.27)
-				)
-			)
-		)
-		(property "Footprint" "Package_DFN_QFN:QFN-24-1EP_5x5mm_P0.65mm_EP3.25x3.25mm"
-			(at 138.43 76.2 0)
-			(hide yes)
-			(show_name no)
-			(do_not_autoplace no)
-			(effects
-				(font
-					(size 1.27 1.27)
-				)
-			)
-		)
-		(property "Datasheet" ""
-			(at 138.43 76.2 0)
-			(hide yes)
-			(show_name no)
-			(do_not_autoplace no)
-			(effects
-				(font
-					(size 1.27 1.27)
-				)
-			)
-		)
-		(property "Description" ""
-			(at 138.43 76.2 0)
-			(hide yes)
-			(show_name no)
-			(do_not_autoplace no)
-			(effects
-				(font
-					(size 1.27 1.27)
-				)
-			)
-		)
-		(pin "17"
-		)
-		(pin "12"
-		)
-		(pin "3"
-		)
-		(pin "13"
-		)
-		(pin "7"
-		)
-		(pin "5"
-		)
-		(pin "1"
-		)
-		(pin "9"
-		)
-		(pin "14"
-		)
-		(pin "10"
-		)
-		(pin "4"
-		)
-		(pin "15"
-		)
-		(pin "6"
-		)
-		(pin "8"
-		)
-		(pin "16"
-		)
-		(pin "2"
-		)
-		(pin "11"
-		)
-		(pin "22"
-		)
-		(pin "18"
-		)
-		(pin "19"
-		)
-		(pin "20"
-		)
-		(pin "21"
-		)
-		(instances
-			(project "avionics-hw27-kiwi-detonator"
-				(path "/297671c8-3551-4118-92b1-deb87cab12e1/0330f3d0-2b5d-4e75-91ab-7f32b2268b09"
-					(reference "U2")
-					(unit 1)
-				)
-			)
-		)
-	)
 )

Commit message: Adding SX1262 symbol
Parts:
- added U2: (no value), Package_DFN_QFN:QFN-24-1EP_5x5mm_P0.65mm_EP3.25x3.25mm, symbol Argus-Miscellaneous:E22-900M30S-SX1262
Changed lines of the file:
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@@
 	(generator_version "10.0")
 	(paper "A4")
+	(symbol
+		(lib_id "Argus-Miscellaneous:E22-900M30S-SX1262")
+		(at 138.43 76.2 0)
+		(unit 1)
+		(body_style 1)
+		(exclude_from_sim no)
+		(in_bom yes)
+		(on_board yes)
+		(in_pos_files yes)
+		(dnp no)
+		(fields_autoplaced yes)
+		(property "Reference" "U2"
+			(at 139.065 77.47 0)
+			(show_name no)
+			(do_not_autoplace no)
+			(effects
+				(font
+					(size 1.27 1.27)
+				)
+			)
+		)
+		(property "Value" ""
+			(at 138.43 76.2 0)
+			(show_name no)
+			(do_not_autoplace no)
+			(effects
+				(font
+					(size 1.27 1.27)
+				)
+			)
+		)
+		(property "Footprint" "Package_DFN_QFN:QFN-24-1EP_5x5mm_P0.65mm_EP3.25x3.25mm"
+			(at 138.43 76.2 0)
+			(hide yes)
+			(show_name no)
+			(do_not_autoplace no)
+			(effects
+				(font
+					(size 1.27 1.27)
+				)
+			)
+		)
+		(property "Datasheet" ""
+			(at 138.43 76.2 0)
+			(hide yes)
+			(show_name no)
+			(do_not_autoplace no)
+			(effects
+				(font
+					(size 1.27 1.27)
+				)
+			)
+		)
+		(property "Description" ""
+			(at 138.43 76.2 0)
+			(hide yes)
+			(show_name no)
+			(do_not_autoplace no)
+			(effects
+				(font
+					(size 1.27 1.27)
+				)
+			)
+		)
+		(pin "17"
+		)
+		(pin "12"
+		)
+		(pin "3"
+		)
+		(pin "13"
+		)
+		(pin "7"
+		)
+		(pin "5"
+		)
+		(pin "1"
+		)
+		(pin "9"
+		)
+		(pin "14"
+		)
+		(pin "10"
+		)
+		(pin "4"
+		)
+		(pin "15"
+		)
+		(pin "6"
+		)
+		(pin "8"
+		)
+		(pin "16"
+		)
+		(pin "2"
+		)
+		(pin "11"
+		)
+		(pin "22"
+		)
+		(pin "18"
+		)
+		(pin "19"
+		)
+		(pin "20"
+		)
+		(pin "21"
+		)
+		(instances
+			(project "avionics-hw27-kiwi-detonator"
+				(path "/297671c8-3551-4118-92b1-deb87cab12e1/0330f3d0-2b5d-4e75-91ab-7f32b2268b09"
+					(reference "U2")
+					(unit 1)
+				)
+			)
+		)
+	)
 )
