File: Detonator_Side/avionics-hw27-kiwi-detonator.kicad_sch (KiCad schematic)
At the start: 0 parts

Commit message: added lower hierarchy schematic files
Other:
- removed sheet Transciever Board
- added sheet Transciever (transciever.kicad_sch)
Changed lines of the file:
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@@
-	)
-	(sheet
-		(at 31.75 34.29)
-		(size 73.66 27.94)
-		(exclude_from_sim no)
-		(in_bom yes)
-		(on_board yes)
-		(dnp no)
-		(fields_autoplaced yes)
-		(stroke
-			(width 0.1524)
-			(type solid)
-		)
-		(fill
-			(color 0 0 0 0)
-		)
-		(property "Sheetname" "Transciever Board"
-			(at 31.75 33.5784 0)
-			(show_name no)
-			(do_not_autoplace no)
-			(effects
-				(font
-					(size 1.27 1.27)
-				)
-				(justify left bottom)
-			)
-		)
-		(property "Sheetfile" "transceiver.kicad_sch"
-			(at 31.75 62.8146 0)
-			(show_name no)
-			(do_not_autoplace no)
-			(effects
-				(font
-					(size 1.27 1.27)
-				)
-				(justify left top)
-			)
-		)
-		(instances
-			(project "avionics-hw27-kiwi-detonator"
-				(path "/297671c8-3551-4118-92b1-deb87cab12e1"
-					(page "2")
-				)
-			)
-		)
 	)
 	(sheet
@@
 				)
 			)
+		)
+	)
+	(sheet
+		(at 31.75 33.02)
+		(size 73.66 27.94)
+		(exclude_from_sim no)
+		(in_bom yes)
+		(on_board yes)
+		(dnp no)
+		(fields_autoplaced yes)
+		(stroke
+			(width 0.1524)
+			(type solid)
+		)
+		(fill
+			(color 0 0 0 0)
+		)
+		(property "Sheetname" "Transciever"
+			(at 31.75 32.3084 0)
+			(show_name no)
+			(do_not_autoplace no)
+			(effects
+				(font
+					(size 1.27 1.27)
+				)
+				(justify left bottom)
+			)
+		)
+		(property "Sheetfile" "transciever.kicad_sch"
+			(at 31.75 61.5446 0)
+			(show_name no)
+			(do_not_autoplace no)
+			(effects
+				(font
+					(size 1.27 1.27)
+				)
+				(justify left top)
+			)
+		)
+		(instances
+			(project "avionics-hw27-kiwi-detonator"
+				(path "/297671c8-3551-4118-92b1-deb87cab12e1"
+					(page "2")
+				)
+			)

Commit message: added microcontroller net and added part to mcu file
Other:
- added sheet Microcontroller (mcu.kicad_sch)
Changed lines of the file:
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@@
 	(paper "A4")
 	(sheet
-		(at 129.54 86.36)
-		(size 77.47 22.86)
+		(at 123.19 72.39)
+		(size 74.93 22.86)
 		(exclude_from_sim no)
 		(in_bom yes)
@@
 		)
 		(property "Sheetname" "RF and Antenna"
-			(at 129.54 85.6484 0)
+			(at 123.19 71.6784 0)
 			(show_name no)
 			(do_not_autoplace no)
@@
 		)
 		(property "Sheetfile" "RF_Antenna.kicad_sch"
-			(at 129.54 109.8046 0)
+			(at 123.19 95.8346 0)
 			(show_name no)
 			(do_not_autoplace no)
@@
 	)
 	(sheet
-		(at 130.81 34.29)
+		(at 123.19 34.29)
 		(size 74.93 26.67)
 		(exclude_from_sim no)
@@
 		)
 		(property "Sheetname" "Detonator"
-			(at 130.81 33.5784 0)
+			(at 123.19 33.5784 0)
 			(show_name no)
 			(do_not_autoplace no)
@@
 		)
 		(property "Sheetfile" "Detonator.kicad_sch"
-			(at 130.81 61.5446 0)
+			(at 123.19 61.5446 0)
 			(show_name no)
 			(do_not_autoplace no)
@@
 	)
 	(sheet
-		(at 102.87 121.92)
-		(size 31.75 21.59)
+		(at 123.19 107.95)
+		(size 76.2 26.67)
 		(exclude_from_sim no)
 		(in_bom yes)
@@
 		)
 		(property "Sheetname" "Speaker"
-			(at 102.87 121.2084 0)
+			(at 123.19 107.2384 0)
 			(show_name no)
 			(do_not_autoplace no)
@@
 		)
 		(property "Sheetfile" "speaker.kicad_sch"
-			(at 102.87 144.0946 0)
+			(at 123.19 135.2046 0)
 			(show_name no)
 			(do_not_autoplace no)
@@
 	)
 	(sheet
-		(at 31.75 85.09)
+		(at 31.75 71.12)
 		(size 72.39 25.4)
 		(exclude_from_sim no)
@@
 		)
 		(property "Sheetname" "Power Supply"
-			(at 31.75 84.3784 0)
+			(at 31.75 70.4084 0)
 			(show_name no)
 			(do_not_autoplace no)
@@
 		)
 		(property "Sheetfile" "Power.kicad_sch"
-			(at 31.75 111.0746 0)
+			(at 31.75 97.1046 0)
 			(show_name no)
 			(do_not_autoplace no)
@@
 				)
 			)
+		)
+	)
+	(sheet
+		(at 31.75 107.95)
+		(size 72.39 25.4)
+		(exclude_from_sim no)
+		(in_bom yes)
+		(on_board yes)
+		(dnp no)
+		(fields_autoplaced yes)
+		(stroke
+			(width 0.1524)
+			(type solid)
+		)
+		(fill
+			(color 0 0 0 0)
+		)
+		(property "Sheetname" "Microcontroller"
+			(at 31.75 107.2384 0)
+			(show_name no)
+			(do_not_autoplace no)
+			(effects
+				(font
+					(size 1.27 1.27)
+				)
+				(justify left bottom)
+			)
+		)
+		(property "Sheetfile" "mcu.kicad_sch"
+			(at 31.75 133.9346 0)
+			(show_name no)
+			(do_not_autoplace no)
+			(effects
+				(font
+					(size 1.27 1.27)
+				)
+				(justify left top)
+			)
+		)
+		(instances
+			(project "avionics-hw27-kiwi-detonator"
+				(path "/297671c8-3551-4118-92b1-deb87cab12e1"
+					(page "7")
+				)
+			)

Commit message: Added RF footprint
Changed lines of the file:
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@@
 	(generator_version "10.0")
 	(paper "A4")
+	(bus
+		(pts
+			(xy 104.14 95.25) (xy 113.03 95.25)
+		)
+		(stroke
+			(width 0)
+			(type default)
+		)
+	)
+	(bus
+		(pts
+			(xy 113.03 95.25) (xy 113.03 113.03)
+		)
+		(stroke
+			(width 0)
+			(type default)
+		)
+	)
+	(bus
+		(pts
+			(xy 113.03 113.03) (xy 104.14 113.03)
+		)
+		(stroke
+			(width 0)
+			(type default)
+		)
+	)
+	(hierarchical_label "Power"
+		(shape input)
+		(at 104.14 95.25 180)
+		(effects
+			(font
+				(size 1.27 1.27)
+			)
+			(justify right)
+		)
+	)
+	(hierarchical_label "Power"
+		(shape input)
+		(at 104.14 113.03 180)
+		(effects
+			(font
+				(size 1.27 1.27)
+			)
+			(justify right)
+		)
+	)
 	(sheet
 		(at 123.19 72.39)
